File: afzuiging/afzuiging-pcb.kicad_pcb (KiCad board)
At the start: 2 copper layers, 70 x 70 mm, 19 parts, among them J1 Voeding, J2 Signaal 1, J3 Signaal 2, U2 ESP32_DevKit_V1_DOIT, U3 L7805, U4 MCP6002-xP

Commit message: Use OpAmp NE5532N
NE5532N can actually be used for 10 volt. MCP6002 has a maximum voltage of 6 volt.
Parts:
- U4: value MCP6002-xP -> NE5532N
Changed lines of the file:
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@@
         (effects (font (size 1 1) (thickness 0.15)))
     )
-    (fp_text value "MCP6002-xP" (at 3.81 9.95) (layer "F.Fab")
+    (fp_text value "NE5532N" (at 3.81 9.95) (layer "F.Fab")
         (effects (font (size 1 1) (thickness 0.15)))
     )
